Commit message: simple controller added

File: src/bumperbot_description/urdf/bumperbot.urdf.xacro (robot description, xacro)
@@ -1,5 +1,8 @@
 <?xml version="1.0"?>
 <robot name="bumperbot" xmlns:xacro="http://www.ros2.org.wiki/xacro" >
-    <xacro:arg name="is_ignition" default="true" />
+    <!-- Start GZ or Ignition depending on ROS 2 Version -->
+    <xacro:arg name="is_ignition" default="true"/>
+    <!-- Load Simulated or Real Hardware Interfaces -->
+    <xacro:arg name="is_sim" default="true"/>
     <!-- Include Gazebo Parameters-->
     <xacro:include filename="$(find bumperbot_description)/urdf/bumperbot_gazebo.xacro" />
@@ -11,14 +14,16 @@
             <origin xyz="0 0 0.04" rpy="0.0 0.25 0.3"/>
             <mass value="8.2573504e-01"/>
-            <inertia ixx="2.2124416e-02" ixy="-1.2294101e-04" ixz="3.4938785e-04" iyy="2.1193702e-02" iyz="-5.0120904e-05" izz="2.0064271e-02"/>
+            <inertia ixx="2.2124416e-02" ixy="-1.2294101e-04" ixz="3.4938785e-04"
+            iyy="2.1193702e-02" iyz="-5.0120904e-05" izz="2.0064271e-02"/>
         </inertial>
         <visual>
-            <origin rpy="0 0 0" xyz="0 0 0"/>
+            <origin xyz="0 0 0" rpy="0 0 0"/>
             <geometry>
                 <mesh filename="package://bumperbot_description/meshes/base_link.STL"/>
             </geometry>
+            <material name="black"/>
         </visual>
         <collision>
-            <origin rpy="0 0 0" xyz="0 0 0"/>
+            <origin xyz="0 0 0" rpy="0 0 0"/>
             <geometry>
                 <mesh filename="package://bumperbot_description/meshes/base_link.STL"/>
@@ -29,5 +34,5 @@
         <parent link="base_footprint"/>
         <child link="base_link"/>
-        <origin rpy="0 0 0" xyz="0 0 0.033"/>
+        <origin xyz="0 0 0.033" rpy="0 0 0"/>
     </joint>
     <link name="wheel_right_link">
@@ -35,11 +40,13 @@
             <origin xyz="0 -0.014 0" rpy="0 0 0"/>
             <mass value="0.0530086090966721"/>
-            <inertia ixx="1.88176298336665E-05" ixy="-4.8444933029987E-10" ixz="1.88163708851143E-08" iyy="3.11510738647764E-05" iyz="-6.93560663069607E-11" izz="1.8801969558182E-05"/>
+            <inertia ixx="1.88176298336665E-05" ixy="-4.8444933029987E-10" ixz="1.88163708851143E-08"
+            iyy="3.11510738647764E-05" iyz="-6.93560663069607E-11" izz="1.8801969558182E-05"/>
         </inertial>
         <visual>
-            <origin rpy="1.57 0 0" xyz="0 0 0" />
+            <origin xyz="0 0 0" rpy="1.57 0 0"/>
             <geometry>
                 <mesh filename="package://bumperbot_description/meshes/wheel_right_link.STL"/>
             </geometry>
+            <material name="blue"/>
         </visual>
         <collision>
@@ -51,8 +58,8 @@
     </link>
     <joint name="wheel_right_joint" type="continuous">
+        <origin xyz="0 -0.0701101849418637 0" rpy="0 0 0"/>
         <parent link="base_link"/>
         <child link="wheel_right_link"/>
         <axis xyz="0 1 0"/>
-        <origin rpy="0 0 0" xyz="0 -0.07 0"/>
     </joint>
     <link name="wheel_left_link">
@@ -60,14 +67,16 @@
             <origin xyz="0 0.014 0" rpy="0 0 0"/>
             <mass value="0.0530086043217644"/>
-            <inertia ixx="1.8792911368909E-05" ixy="3.31256392204584E-10" ixz="-1.14082001662767E-08" iyy="3.11510738759073E-05" iyz="-3.60499245082192E-10" izz="1.88266886146847E-05"/>
+            <inertia ixx="1.8792911368909E-05" ixy="3.31256392204584E-10" ixz="-1.14082001662767E-08"
+            iyy="3.11510738759073E-05" iyz="-3.60499245082192E-10" izz="1.88266886146847E-05"/>
         </inertial>
         <visual>
-            <origin rpy="-1.57 0 0" xyz="0 0 0" />
+            <origin xyz="0 0 0" rpy="-1.57 0 0"/>
             <geometry>
                 <mesh filename="package://bumperbot_description/meshes/wheel_left_link.STL"/>
             </geometry>
+            <material name="blue"/>
         </visual>
         <collision>
-            <origin xyz="0 0.015 0" rpy="1.57 0 0"/>
+            <origin xyz="0 0.015 0" rpy="-1.57 0 0"/>
             <geometry>
                 <sphere radius="0.033" />
@@ -76,8 +85,8 @@
     </link>
     <joint name="wheel_left_joint" type="continuous">
+        <origin xyz="0 0.0701101849418642 0" rpy="0 0 0"/>
         <parent link="base_link"/>
         <child link="wheel_left_link"/>
         <axis xyz="0 1 0"/>
-        <origin rpy="0 0 0" xyz="0 0.07 0"/>
     </joint>
     <link name="caster_front_link">
@@ -88,8 +97,9 @@
         </inertial>
         <visual>
-        <origin rpy="0 0 0" xyz="0 0 0"/>
+        <origin xyz="0 0 0" rpy="0 0 0"/>
             <geometry>
                 <mesh filename="package://bumperbot_description/meshes/caster_front_link.STL"/>
             </geometry>
+            <material name="silver"/>
         </visual>
         <collision>
@@ -103,5 +113,5 @@
         <parent link="base_link"/>
         <child link="caster_front_link"/>
-        <origin rpy="0 0 0" xyz="0.04755 0 -0.0275"/>
+        <origin xyz="0.04755 0 -0.0275" rpy="0 0 0"/>
     </joint>
     <link name="caster_rear_link">
@@ -109,11 +119,14 @@
             <origin xyz="3.8996812895542E-07 2.40073004698083E-07 0.00219173397061509" rpy="0 0 0"/>
             <mass value="1.44379265037902E-06"/>
-            <inertia ixx="7.23075276010246E-11" ixy="-6.10956872363424E-16" ixz="2.22849693527207E-15" iyy="3.87137930859167E-11" iyz="2.939098587861E-15" izz="1.00967486676306E-10"/>
+            <inertia ixx="7.23075276010246E-11" ixy="-6.10956872363424E-16" ixz="2.22849693527207E-15"
+             iyy="3.87137930859167E-11" iyz="2.939098587861E-15"
+             izz="1.00967486676306E-10"/>
         </inertial>
         <visual>
-        <origin rpy="0 0 0" xyz="0 0 0"/>
+        <origin xyz="0 0 0" rpy="0 0 0"/>
             <geometry>
                 <mesh filename="package://bumperbot_description/meshes/caster_rear_link.STL"/>
             </geometry>
+            <material name="silver"/>
         </visual>
         <collision>
@@ -125,7 +138,8 @@
     </link>
     <joint name="caster_rear_joint" type="fixed">
+        <origin xyz="-0.04755 0 -0.0275" rpy="0 0 0"/>
         <parent link="base_link"/>
         <child link="caster_rear_link"/>
-        <origin rpy="0 0 0" xyz="-0.04755 0 -0.0275"/>
+        <axis xyz="0 0 0" />
     </joint>
 </robot>

File: src/bumperbot_description/urdf/bumperbot_gazebo.xacro (robot description, xacro)
@@ -25,5 +25,5 @@
         <kd>100</kd>
         <minDepth>0.001</minDepth>
-        <maxVel>0.1</maxVel>
+        <maxVel>1.0</maxVel>
     </gazebo>
     <gazebo reference="caster_rear_link">
@@ -33,5 +33,5 @@
         <kd>100</kd>
         <minDepth>0.001</minDepth>
-        <maxVel>0.1</maxVel>
+        <maxVel>1.0</maxVel>
     </gazebo>
     <gazebo>
